Commit message: add: STL mesh file for visualization, macros for mass & inertia values

File: ros2_ws/src/simulator_description/urdf/racecar.xacro (robot description, xacro)
@@ -1,148 +1,44 @@
 <?xml version="1.0"?>
 <robot xmlns:xacro="http://www.ros.org/wiki/xacro"  name="robot">
-    <!-- This first link called "world" is empty -->
+    <xacro:property name="RACECAR_WIDTH" value="1.575"/>
+    <xacro:property name="RACECAR_LENGTH" value="2.5"/>
+    <xacro:property name="RACECAR_HEIGHT" value="1.4"/>
+    <xacro:property name="COG_HEIGHT" value="0.7"/>
+    <xacro:property name="RACECAR_COLLISION_STL" value="file://$(find simulator_description)/meshes/whole_car.stl"/>
+    <xacro:property name="RACECAR_VISUAL_DAE" value=""/>
+    <xacro:property name="RACECAR_MASS" value="190.0"/> <!-- Mass in KG -->
+    <xacro:property name="RACECAR_INERTIA_IXX" value="2.26"/>
+    <xacro:property name="RACECAR_INERTIA_IXY" value="0.0"/>
+    <xacro:property name="RACECAR_INERTIA_IXZ" value="0.0"/>
+    <xacro:property name="RACECAR_INERTIA_IYY" value="6.26"/>
+    <xacro:property name="RACECAR_INERTIA_IYZ" value="0.0"/>
+    <xacro:property name="RACECAR_INERTIA_IZZ" value="8.5"/>
+    <material name="blue"> <color rgba="0.0 0.0 1.0 0.5"/>  </material>
+    <material name="orange"> <color rgba="1.0 1.0 0.0 0.5"/>  </material>
+    <material name="white"> <color rgba="1.0 1.0 1.0 0.5"/>  </material>
+    <material name="black"> <color rgba="0.0 0.0 0.0 0.9"/>  </material>
+    <link name="base_footprint">
+    </link>
+    <joint name="base_footprint_to_base_chassis" type="fixed">
+        <origin xyz="0.0 0.0 0.0"/> <!-- COG_HEIGHT-->
+        <parent link="base_footprint"/>
+        <child link="base_chassis" />
+    </joint>
     <link name="base_chassis">
-    </link>
-    <!-- A simple fixed joint from our empty world link, to our base. -->
-    <!-- The base origin is offset from the world origin. -->
-    <joint name="base_joint" type="fixed">
-        <origin xyz="1.5 1.0 0" rpy="0 0 0"/>
-        <parent link="base_chassis"/>
-        <child link="base_link"/>
-    </joint>
-    <!-- base_link is a large rectangular plate. Some things to note: -->
-    <!-- - We set the visual origin Z to half the box height, so that the link origin sits at the bottom of the box -->
-    <!-- - We set the collision to be identical to the visual -->
-    <!-- - We specified the colour manually (but still need to enter a name) -->
-    <!-- - We specified all the inertial parameters manually -->
-    <link name="base_link">
         <visual>
-            <origin xyz="0 0 0.05" rpy="0 0 0"/>
             <geometry>
-                <box size="2.5 1.5 0.1" />
+                <!-- scaled because STL model is really strange-->
+                <mesh filename="${RACECAR_COLLISION_STL}" scale="0.001 0.001 0.001"/>
             </geometry>
-            <material name="green">
-                <color rgba="0.2 1 0.2 1"/>
-            </material>
+            <material name="black" />
         </visual>
         <collision>
-            <origin xyz="0 0 0.05" rpy="0 0 0"/>
             <geometry>
-                <box size="2.5 1.5 0.1" />
+                <mesh filename="${RACECAR_COLLISION_STL}" scale="0.001 0.001 0.001"/>
             </geometry>
         </collision>
         <inertial>
-            <origin xyz="0 0 0.05" rpy="0 0 0"/>
-            <mass value="12" />
-            <inertia ixx="2.26" ixy="0.0" ixz="0.0" iyy="6.26" iyz="0.0" izz="8.5" />
-        </inertial>
-    </link>
-    <!-- slider_joint lets slider_link move back and forth along the top of the base in one dimension.  -->
-    <!-- - Origin is set to one of the top edges of the base_link box, so that our link skims across the top  -->
-    <!-- - It moves along the X axis -->
-    <!-- - We need to specify limits for the motion -->
-    <joint name="slider_joint" type="prismatic">
-        <origin xyz="-1.25 0 0.1" rpy="0 0 0"/>
-        <parent link="base_link"/>
-        <child link="slider_link"/>
-        <axis xyz="1 0 0"/>
-        <limit lower="0" upper="2" velocity="100" effort="100"/>
-    </joint>
-    <!-- slider_link is the box skimming across the top of the base. Its parameters are similar to the base_link, however: -->
-    <!-- - Instead of explicitly describing a colour, it uses the named material "blue". It knows about "blue" that material was included in example_include.xacro. -->
-    <!-- - Instead of explicitly describing the inertia, we use a macro that was defined in the example_include.xacro -->
-    <link name="slider_link">
-        <visual>
-            <origin xyz="0 0 0.075" rpy="0 0 0"/>
-            <geometry>
-                <box size="0.5 0.25 0.15" />
-            </geometry>
-            <material name="blue" />
-        </visual>
-        <collision>
-            <origin xyz="0 0 0.075" rpy="0 0 0"/>
-            <geometry>
-                <box size="0.5 0.25 0.15" />
-            </geometry>
-        </collision>
-        <inertial>
-            <origin xyz="0 0 0.05" rpy="0 0 0"/>
-            <mass value="12" />
-            <inertia ixx="2.26" ixy="0.0" ixz="0.0" iyy="6.26" iyz="0.0" izz="8.5" />
-        </inertial>
-    </link>
-    <!-- arm_joint describes the rotation of the arm and is centred around the top corner of the slider box. -->
-    <!-- - The axis of rotation is -1 in Y, so that positive is "up" -->
-    <!-- - The upper limit uses xacro's mathematical features -->
-    <joint name="arm_joint" type="revolute">
-        <origin xyz="0.25 0 0.15" rpy="0 0 0"/>
-        <parent link="slider_link"/>
-        <child link="arm_link"/>
-        <axis xyz="0 -1 0"/>
-        <limit lower="0" upper="${pi/2}" velocity="100" effort="100"/>
-    </joint>
-    <!-- arm_link describes the arm -->
-    <!-- - We use the "property" feature to define the arm length and radius and use them multiple times -->
-    <!-- - The visual/collision origin is set to halfway along the length (similar to the box), but also with a rotation (again using the mathematical features). -->
-    <!--   This is because the cylinder extends along the Z axis by default, but we want it to be along the X axis (when the joint is at 0) -->
-    <xacro:property name="arm_length" value="1" />
-    <xacro:property name="arm_radius" value="0.1" />
-    <link name="arm_link">
-        <visual>
-            <origin xyz="${arm_length/2} 0 0" rpy="0 ${pi/2} 0"/>
-            <geometry>
-                <cylinder length="${arm_length}" radius="${arm_radius}" />
-            </geometry>
-            <material name="orange" />
-        </visual>
-        <collision>
-            <origin xyz="${arm_length/2} 0 0" rpy="0 ${pi/2} 0"/>
-            <geometry>
-                <cylinder length="${arm_length}" radius="${arm_radius}" />
-            </geometry>
-        </collision>
-        <inertial>
-            <origin xyz="0 0 0.05" rpy="0 0 0"/>
-            <mass value="12" />
-            <inertia ixx="2.26" ixy="0.0" ixz="0.0" iyy="6.26" iyz="0.0" izz="8.5" />
-        </inertial>
-    </link>
-    <!-- camera_joint describes where the camera is relative to the arm -->
-    <!-- - Even though the camera isn't moving relative to the arm, it will probably be helpful to have its own link/frame rather than just adding more visuals to the arm -->
-    <!-- - For this example, the camera_link origin will be at the centre of the camera's "sensor" -->
-    <joint name="camera_joint" type="fixed">
-        <origin xyz="${arm_length} 0 ${arm_radius + 0.075}" rpy="0 0 0"/>
-        <parent link="arm_link"/>
-        <child link="camera_link"/>
-    </joint>
-    <!-- camera_link describes the camera at the end of the arm -->
-    <!-- - It has multiple visual elements, which ultimately get combined together -->
-    <!-- - Even if we specify different materials, RViz will just colour them all the same as the first -->
-    <!-- - Although we could also specify multiple collision geometries, instead we just use a single box that encompasses the whole camera -->
-    <link name="camera_link">
-        <visual>
-            <origin xyz="-0.03 0 0" rpy="0 0 0"/>
-            <geometry>
-                <box size="0.06 0.15 0.15" />
-            </geometry>
-            <material name="white" />
-        </visual>
-        <visual>
-            <origin xyz="0.03 0 0" rpy="0 ${pi/2} 0"/>
-            <geometry>
-                <cylinder length="0.06" radius="0.04" />
-            </geometry>
-            <material name="blue" />
-        </visual>
-        <collision>
-            <origin xyz="0.0 0 0" rpy="0 0 0"/>
-            <geometry>
-                <box size="0.12 0.15 0.15" />
-            </geometry>
-        </collision>
-        <inertial>
-            <origin xyz="0 0 0.05" rpy="0 0 0"/>
-            <mass value="12" />
-            <inertia ixx="2.26" ixy="0.0" ixz="0.0" iyy="6.26" iyz="0.0" izz="8.5" />
+            <mass value="${RACECAR_MASS}" />
+            <inertia ixx="${RACECAR_INERTIA_IXX}" ixy="${RACECAR_INERTIA_IXY}" ixz="${RACECAR_INERTIA_IXZ}" iyy="${RACECAR_INERTIA_IYY}" iyz="${RACECAR_INERTIA_IYZ}" izz="${RACECAR_INERTIA_IZZ}" />
         </inertial>
     </link>

Commit message: add: joints & wheels to be tested

File: ros2_ws/src/simulator_description/urdf/racecar.xacro (robot description, xacro)
@@ -1,10 +1,14 @@
 <?xml version="1.0"?>
 <robot xmlns:xacro="http://www.ros.org/wiki/xacro"  name="robot">
+    <!-- STL & DAE files -->
+    <xacro:property name="RACECAR_WHEEL_STL" value="file://$(find simulator_description)/meshes/wheel.stl"/>
+    <xacro:property name="RACECAR_COLLISION_STL" value="file://$(find simulator_description)/meshes/whole_car.stl"/>
+    <xacro:property name="RACECAR_VISUAL_DAE" value=""/>
+    <xacro:property name="RACECAR_STEERING_HINGE_STL" value="file://$(find simulator_description)/meshes/steering_hinge.stl"/>
+    <!-- Vehicle Dynamics & So on -->
     <xacro:property name="RACECAR_WIDTH" value="1.575"/>
     <xacro:property name="RACECAR_LENGTH" value="2.5"/>
     <xacro:property name="RACECAR_HEIGHT" value="1.4"/>
     <xacro:property name="COG_HEIGHT" value="0.7"/>
-    <xacro:property name="RACECAR_COLLISION_STL" value="file://$(find simulator_description)/meshes/whole_car.stl"/>
-    <xacro:property name="RACECAR_VISUAL_DAE" value=""/>
     <xacro:property name="RACECAR_MASS" value="190.0"/> <!-- Mass in KG -->
     <xacro:property name="RACECAR_INERTIA_IXX" value="2.26"/>
@@ -14,4 +18,5 @@
     <xacro:property name="RACECAR_INERTIA_IYZ" value="0.0"/>
     <xacro:property name="RACECAR_INERTIA_IZZ" value="8.5"/>
+    <xacro:property name="DUMMY_VALUE" value="0.0" />
     <material name="blue"> <color rgba="0.0 0.0 1.0 0.5"/>  </material>
     <material name="orange"> <color rgba="1.0 1.0 0.0 0.5"/>  </material>
@@ -43,3 +48,138 @@
         </inertial>
     </link>
+    <joint name="base_chassis_to_steering_hinge" type="revolute">
+        <parent link="base_chassis"/>
+        <child link="steering_hinge" />
+        <axis>
+            <xyz expressed_in='__model__'>0 1 0</xyz>
+            <limit>
+                <lower>-1.79769e+308</lower>    <!--negative infinity-->
+                <upper>1.79769e+308</upper>     <!--positive infinity-->
+            </limit>
+        </axis>
+    </joint>
+    <link name="steering_hinge">
+        <visual>
+            <geometry>
+                <mesh filename="${RACECAR_STEERING_HINGE_STL}" scale="0.001 0.001 0.001"/>
+            </geometry>
+        </visual>
+        <collision>
+            <geometry>
+                <mesh filename="${RACECAR_STEERING_HINGE_STL}" scale="0.001 0.001 0.001"/>
+            </geometry>
+        </collision>
+        <inertial>
+            <mass value="${DUMMY_VALUE}"/>
+            <inertia ixx="${DUMMY_VALUE}" ixy="${DUMMY_VALUE}" ixz="${DUMMY_VALUE}" iyy="${DUMMY_VALUE}" iyz="${DUMMY_VALUE}" izz="${DUMMY_VALUE}"/>
+        </inertial>
+    </link>
+    <joint name="steering_hinge_to_left_front_wheel" type="revolute">
+        <parent link="steering_hinge"/>
+        <child link="left_front_wheel" />
+        <axis>
+            <xyz expressed_in='__model__'>0 1 0</xyz>
+            <limit>
+                <lower>-1.79769e+308</lower>    <!--negative infinity-->
+                <upper>1.79769e+308</upper>     <!--positive infinity-->
+            </limit>
+        </axis>
+    </joint>
+    <link name="left_front_wheel">
+        <visual>
+            <geometry>
+                <mesh filename="${RACECAR_WHEEL_STL}" scale="0.001 0.001 0.001"/>
+            </geometry>
+        </visual>
+        <collision>
+            <geometry>
+                <mesh filename="${RACECAR_WHEEL_STL}" scale="0.001 0.001 0.001"/>
+            </geometry>
+        </collision>
+        <inertial>
+            <mass value="${DUMMY_VALUE}"/>
+            <inertia ixx="${DUMMY_VALUE}" ixy="${DUMMY_VALUE}" ixz="${DUMMY_VALUE}" iyy="${DUMMY_VALUE}" iyz="${DUMMY_VALUE}" izz="${DUMMY_VALUE}"/>
+        </inertial>
+    </link>
+    <joint name="steering_hinge_to_right_front_wheel" type="revolute">
+        <parent link="steering_hinge"/>
+        <child link="right_front_wheel" />
+        <axis>
+            <xyz expressed_in='__model__'>0 1 0</xyz>
+            <limit>
+                <lower>-1.79769e+308</lower>    <!--negative infinity-->
+                <upper>1.79769e+308</upper>     <!--positive infinity-->
+            </limit>
+        </axis>
+    </joint>
+    <link name="right_front_wheel">
+        <visual>
+            <geometry>
+                <mesh filename="${RACECAR_WHEEL_STL}" scale="0.001 0.001 0.001"/>
+            </geometry>
+        </visual>
+        <collision>
+            <geometry>
+                <mesh filename="${RACECAR_WHEEL_STL}" scale="0.001 0.001 0.001"/>
+            </geometry>
+        </collision>
+        <inertial>
+            <mass value="${DUMMY_VALUE}"/>
+            <inertia ixx="${DUMMY_VALUE}" ixy="${DUMMY_VALUE}" ixz="${DUMMY_VALUE}" iyy="${DUMMY_VALUE}" iyz="${DUMMY_VALUE}" izz="${DUMMY_VALUE}"/>
+        </inertial>
+    </link>
+    <joint name="base_chassis_to_left_rear_wheel" type="revolute">
+        <parent link="base_chassis"/>
+        <child link="left_rear_wheel" />
+        <axis>
+            <xyz expressed_in='__model__'>0 1 0</xyz>
+            <limit>
+                <lower>-1.79769e+308</lower>    <!--negative infinity-->
+                <upper>1.79769e+308</upper>     <!--positive infinity-->
+            </limit>
+        </axis>
+    </joint>
+    <link name="left_rear_wheel">
+        <visual>
+            <geometry>
+                <mesh filename="${RACECAR_WHEEL_STL}" scale="0.001 0.001 0.001"/>
+            </geometry>
+        </visual>
+        <collision>
+            <geometry>
+                <mesh filename="${RACECAR_WHEEL_STL}" scale="0.001 0.001 0.001"/>
+            </geometry>
+        </collision>
+        <inertial>
+            <mass value="${DUMMY_VALUE}"/>
+            <inertia ixx="${DUMMY_VALUE}" ixy="${DUMMY_VALUE}" ixz="${DUMMY_VALUE}" iyy="${DUMMY_VALUE}" iyz="${DUMMY_VALUE}" izz="${DUMMY_VALUE}"/>
+        </inertial>
+    </link>
+    <joint name="base_chassis_to_right_rear_wheel" type="revolute">
+        <parent link="base_chassis"/>
+        <child link="right_rear_wheel" />
+        <axis>
+            <xyz expressed_in='__model__'>0 1 0</xyz>
+            <limit>
+                <lower>-1.79769e+308</lower>    <!--negative infinity-->
+                <upper>1.79769e+308</upper>     <!--positive infinity-->
+            </limit>
+        </axis>
+    </joint>
+    <link name="right_rear_wheel">
+        <visual>
+            <geometry>
+                <mesh filename="${RACECAR_WHEEL_STL}" scale="0.001 0.001 0.001"/>
+            </geometry>
+        </visual>
+        <collision>
+            <geometry>
+                <mesh filename="${RACECAR_WHEEL_STL}" scale="0.001 0.001 0.001"/>
+            </geometry>
+        </collision>
+        <inertial>
+            <mass value="${DUMMY_VALUE}"/>
+            <inertia ixx="${DUMMY_VALUE}" ixy="${DUMMY_VALUE}" ixz="${DUMMY_VALUE}" iyy="${DUMMY_VALUE}" iyz="${DUMMY_VALUE}" izz="${DUMMY_VALUE}"/>
+        </inertial>
+    </link>
 </robot>
