Commit message: fix: implemented gazebo's ackermann, now the car moves with a command. removed ros2 control, to be investigated in the future

File: ros2_ws/src/simulator_description/urdf/racecar_control.xacro (robot description, xacro)
@@ -14,8 +14,8 @@
     <xacro:property name="RACECAR_STEERING_HINGE_X" value="0.050"/> <!-- [m] -->
     <xacro:property name="RACECAR_STEERING_HINGE_Y" value="0.575"/> <!-- [m] -->
-    <xacro:property name="RACECAR_STEERING_HINGE_Z" value="0.23"/> <!-- [m] -->
+    <xacro:property name="RACECAR_STEERING_HINGE_Z" value="0.25"/> <!-- [m] -->
     <xacro:property name="RACECAR_WHEEL_REAR_X" value="-1.6" /> <!-- [m] -->
     <xacro:property name="RACECAR_WHEEL_REAR_Y" value="0.575" /> <!-- [m] -->
-    <xacro:property name="RACECAR_WHEEL_REAR_Z" value="0.23" /> <!-- [m] -->
+    <xacro:property name="RACECAR_WHEEL_REAR_Z" value="0.25" /> <!-- [m] -->
     <!-- Racecar Parameters -->
     <!-- most of these parameters depend on the specifics of your vehicle -->
@@ -23,5 +23,5 @@
     <!-- Gazebo wants coherent values for Inertia. -->
     <!-- Consider using the scripts for plugging these values. -->
-    <xacro:property name="RACECAR_WIDTH" value="1.575"/> <!-- [m] -->
+    <xacro:property name="RACECAR_WIDTH" value="0.85"/> <!-- [m] -->
     <xacro:property name="RACECAR_LENGTH" value="2.942"/> <!-- [m] -->
     <xacro:property name="RACECAR_HEIGHT" value="1.119"/> <!-- [m] -->
@@ -50,10 +50,10 @@
     <xacro:property name="WHEEL_HEIGHT" value="0.46" /> <!-- [m] -->
     <xacro:property name="WHEEL_MASS" value="10.0"/> <!-- [kg] -->
-    <xacro:property name="WHEEL_INERTIA_IXX" value="0.17633" /> <!-- [kg^2 m] -->
+    <xacro:property name="WHEEL_INERTIA_IXX" value="0.22042" /> <!-- [kg^2 m] -->
     <xacro:property name="WHEEL_INERTIA_IXY" value="0.0" /> <!-- [kg^2 m] -->
     <xacro:property name="WHEEL_INERTIA_IXZ" value="0.0" /> <!-- [kg^2 m] -->
-    <xacro:property name="WHEEL_INERTIA_IYY" value="0.00333" /> <!-- [kg^2 m] -->
+    <xacro:property name="WHEEL_INERTIA_IYY" value="0.26450" /> <!-- [kg^2 m] -->
     <xacro:property name="WHEEL_INERTIA_IYZ" value="0.0" /> <!-- [kg^2 m] -->
-    <xacro:property name="WHEEL_INERTIA_IZZ" value="0.00333" /> <!-- [kg^2 m] -->
+    <xacro:property name="WHEEL_INERTIA_IZZ" value="0.22042" /> <!-- [kg^2 m] -->
     <!-- Actuators Parameters-->
     <xacro:property name="DUMMY_VALUE" value="1.0" />
@@ -84,5 +84,6 @@
             <material name="green" />
         </visual>
-        <collision>
+         <collision>
+            <origin xyz="-0.55 0 0.65"/>
             <geometry>
                 <box size="${RACECAR_LENGTH} ${RACECAR_WIDTH} ${RACECAR_HEIGHT}" />
@@ -136,5 +137,5 @@
         <inertial>
             <mass value="${STEERING_HINGE_MASS}"/>
-            <inertia ixx="${RACECAR_INERTIA_IXX}" ixy="${RACECAR_INERTIA_IXY}" ixz="${RACECAR_INERTIA_IXZ}" iyy="${RACECAR_INERTIA_IYY}" iyz="${RACECAR_INERTIA_IYZ}" izz="${RACECAR_INERTIA_IZZ}" />
+            <inertia ixx="${STEERING_HINGE_INERTIA_IXX}" ixy="${STEERING_HINGE_INERTIA_IXY}" ixz="${STEERING_HINGE_INERTIA_IXZ}" iyy="${STEERING_HINGE_INERTIA_IYY}" iyz="${STEERING_HINGE_INERTIA_IYZ}" izz="${STEERING_HINGE_INERTIA_IZZ}" />
         </inertial>
     </link>
@@ -152,6 +153,5 @@
         <inertial>
             <mass value="${STEERING_HINGE_MASS}"/>
-            <inertia ixx="${RACECAR_INERTIA_IXX}" ixy="${RACECAR_INERTIA_IXY}" ixz="${RACECAR_INERTIA_IXZ}" iyy="${RACECAR_INERTIA_IYY}" iyz="${RACECAR_INERTIA_IYZ}" izz="${RACECAR_INERTIA_IZZ}" />
-        </inertial>
+            <inertia ixx="${STEERING_HINGE_INERTIA_IXX}" ixy="${STEERING_HINGE_INERTIA_IXY}" ixz="${STEERING_HINGE_INERTIA_IXZ}" iyy="${STEERING_HINGE_INERTIA_IYY}" iyz="${STEERING_HINGE_INERTIA_IYZ}" izz="${STEERING_HINGE_INERTIA_IZZ}" />        </inertial>
     </link>
     <joint name="left_steering_hinge_to_left_front_wheel" type="continuous">
@@ -178,11 +178,12 @@
         </visual>
         <collision>
-            <geometry>
-                <box size="${WHEEL_LENGTH} ${WHEEL_WIDTH} ${WHEEL_HEIGHT}"/>
-            </geometry>
-        </collision>
-        <inertial>
-            <mass value="${WHEEL_MASS}"/>
-            <inertia ixx="${RACECAR_INERTIA_IXX}" ixy="${RACECAR_INERTIA_IXY}" ixz="${RACECAR_INERTIA_IXZ}" iyy="${RACECAR_INERTIA_IYY}" iyz="${RACECAR_INERTIA_IYZ}" izz="${RACECAR_INERTIA_IZZ}" />
+            <origin rpy="1.5708 0 0"/>
+            <geometry>
+                <cylinder length="${WHEEL_WIDTH}" radius="${WHEEL_WIDTH}"/>
+            </geometry>
+        </collision>
+        <inertial>
+            <mass value="${WHEEL_MASS}"/>
+            <inertia ixx="${WHEEL_INERTIA_IXX}" ixy="${WHEEL_INERTIA_IXY}" ixz="${WHEEL_INERTIA_IXZ}" iyy="${WHEEL_INERTIA_IYY}" iyz="${WHEEL_INERTIA_IYZ}" izz="${WHEEL_INERTIA_IZZ}" />
         </inertial>
     </link>
@@ -195,11 +196,12 @@
         </visual>
         <collision>
-            <geometry>
-                <box size="${WHEEL_LENGTH} ${WHEEL_WIDTH} ${WHEEL_HEIGHT}"/>
-            </geometry>
-        </collision>
-        <inertial>
-            <mass value="${WHEEL_MASS}"/>
-            <inertia ixx="${RACECAR_INERTIA_IXX}" ixy="${RACECAR_INERTIA_IXY}" ixz="${RACECAR_INERTIA_IXZ}" iyy="${RACECAR_INERTIA_IYY}" iyz="${RACECAR_INERTIA_IYZ}" izz="${RACECAR_INERTIA_IZZ}" />
+            <origin rpy="1.5708 0 0"/>
+            <geometry>
+                <cylinder length="${WHEEL_WIDTH}" radius="${WHEEL_WIDTH}"/>
+            </geometry>
+        </collision>
+        <inertial>
+            <mass value="${WHEEL_MASS}"/>
+            <inertia ixx="${WHEEL_INERTIA_IXX}" ixy="${WHEEL_INERTIA_IXY}" ixz="${WHEEL_INERTIA_IXZ}" iyy="${WHEEL_INERTIA_IYY}" iyz="${WHEEL_INERTIA_IYZ}" izz="${WHEEL_INERTIA_IZZ}" />
         </inertial>
     </link>
@@ -212,12 +214,15 @@
             <material name="black" />
         </visual>
-        <collision>
-            <geometry>
-                <box size="${WHEEL_LENGTH} ${WHEEL_WIDTH} ${WHEEL_HEIGHT}"/>
-            </geometry>
-        </collision>
-        <inertial>
-            <mass value="${WHEEL_MASS}"/>
-            <inertia ixx="${RACECAR_INERTIA_IXX}" ixy="${RACECAR_INERTIA_IXY}" ixz="${RACECAR_INERTIA_IXZ}" iyy="${RACECAR_INERTIA_IYY}" iyz="${RACECAR_INERTIA_IYZ}" izz="${RACECAR_INERTIA_IZZ}" />
+        <collision  name="left_rear_wheel_collision">
+            <origin rpy="1.5708 0 0"/>
+            <geometry>
+                <cylinder
+                    length="${WHEEL_WIDTH}"
+                    radius="${WHEEL_HEIGHT / 2}"/>
+            </geometry>
+        </collision>
+        <inertial>
+            <mass value="${WHEEL_MASS}"/>
+            <inertia ixx="${WHEEL_INERTIA_IXX}" ixy="${WHEEL_INERTIA_IXY}" ixz="${WHEEL_INERTIA_IXZ}" iyy="${WHEEL_INERTIA_IYY}" iyz="${WHEEL_INERTIA_IYZ}" izz="${WHEEL_INERTIA_IZZ}" />
         </inertial>
     </link>
@@ -229,57 +234,38 @@
             <material name="black" />
         </visual>
-        <collision>
-            <geometry>
-                <box size="${WHEEL_LENGTH} ${WHEEL_WIDTH} ${WHEEL_HEIGHT}"/>
-            </geometry>
-        </collision>
-        <inertial>
-            <mass value="${WHEEL_MASS}"/>
-            <inertia ixx="${RACECAR_INERTIA_IXX}" ixy="${RACECAR_INERTIA_IXY}" ixz="${RACECAR_INERTIA_IXZ}" iyy="${RACECAR_INERTIA_IYY}" iyz="${RACECAR_INERTIA_IYZ}" izz="${RACECAR_INERTIA_IZZ}" />
-        </inertial>
-    </link>
-    <!-- ROS2 CONTROL STUFF -->
+        <collision name="right_rear_wheel_collision">
+            <origin rpy="1.5708 0 0"/>
+            <geometry>
+                <cylinder
+                    length="${WHEEL_WIDTH}"
+                    radius="${WHEEL_HEIGHT / 2}"/>
+            </geometry>
+        </collision>
+        <inertial>
+            <mass value="${WHEEL_MASS}"/>
+            <inertia ixx="${WHEEL_INERTIA_IXX}" ixy="${WHEEL_INERTIA_IXY}" ixz="${WHEEL_INERTIA_IXZ}" iyy="${WHEEL_INERTIA_IYY}" iyz="${WHEEL_INERTIA_IYZ}" izz="${WHEEL_INERTIA_IZZ}" />
+        </inertial>
+    </link>
     <gazebo>
-        <plugin filename="libgz_ros2_control-system.so" name="gz_ros2_control::GazeboSimROS2ControlPlugin">
-            <parameters>$(find simulator_description)/config/ackermann_controller_param.yaml</parameters>
-            <controller_manager_name>racecar_controller</controller_manager_name>
-        </plugin>
+        <plugin
+            filename="gz-sim-ackermann-steering-system"
+            name="gz::sim::systems::AckermannSteering">
+            <left_joint>base_chassis_to_left_front_wheel</left_joint>
+            <left_joint>base_chassis_to_left_rear_wheel</left_joint>
+            <right_joint>base_chassis_to_right_front_wheel</right_joint>
+            <right_joint>base_chassis_to_right_rear_wheel</right_joint>
+            <left_steering_joint>base_chassis_to_left_steering_hinge</left_steering_joint>
+            <right_steering_joint>base_chassis_to_right_steering_hinge</right_steering_joint>
+            <kingpin_width>1.0</kingpin_width>
+            <steering_limit>0.5</steering_limit>
+            <wheel_base>1.0</wheel_base>
+            <wheel_separation>1.25</wheel_separation>
+            <wheel_radius>0.3</wheel_radius>
+            <min_velocity>-1</min_velocity>
+            <max_velocity>1</max_velocity>
+            <min_acceleration>-3</min_acceleration>
+            <max_acceleration>3</max_acceleration>
+            <topic>/cmd_vel</topic>
+      </plugin>
     </gazebo>
-    <ros2_control name="RaceCarControl" type="system">
-        <hardware>
-            <plugin>gz_ros2_control/GazeboSimSystem</plugin>
-        </hardware>
-        <joint name="base_chassis_to_left_steering_hinge">
-            <command_interface name="position"/>
-            <state_interface name="velocity"/>
-            <state_interface name="effort"/>
-            <state_interface name="position"/>
-        </joint>
-        <joint name="base_chassis_to_right_steering_hinge">
-            <command_interface name="position"/>
-            <state_interface name="velocity"/>
-            <state_interface name="effort"/>
-            <state_interface name="position"/>
-        </joint>
-        <joint name="base_chassis_to_left_rear_wheel">
-            <command_interface name="velocity"/>
-            <state_interface name="velocity"/>
-            <state_interface name="effort"/>
-        </joint>
-        <joint name="base_chassis_to_right_rear_wheel">
-            <command_interface name="velocity"/>
-            <state_interface name="velocity"/>
-            <state_interface name="effort"/>
-        </joint>
-        <joint name="left_steering_hinge_to_left_front_wheel">
-            <command_interface name="position"/>
-            <state_interface name="velocity"/>
-            <state_interface name="effort"/>
-        </joint>
-        <joint name="right_steering_hinge_to_right_front_wheel">
-            <command_interface name="position"/>
-            <state_interface name="velocity"/>
-            <state_interface name="effort"/>
-        </joint>
-    </ros2_control>
 </robot>

Commit message: style: added macros for variables, no naked numbers in xacro anymore

File: ros2_ws/src/simulator_description/urdf/racecar_control.xacro (robot description, xacro)
@@ -56,6 +56,15 @@
     <xacro:property name="WHEEL_INERTIA_IYZ" value="0.0" /> <!-- [kg^2 m] -->
     <xacro:property name="WHEEL_INERTIA_IZZ" value="0.22042" /> <!-- [kg^2 m] -->
-    <!-- Actuators Parameters-->
-    <xacro:property name="DUMMY_VALUE" value="1.0" />
+    <!-- Gazebo Ackermann Stuff + Joint Limits-->
+    <xacro:property name="RACECAR_STEERING_HINGES_DISTANCE" value="1.15"/> <!-- [m], equal to the kingpin width, distance between steering hinges -->
+    <xacro:property name="MIN_VELOCITY" value="-1"/> <!-- [m/s] -->
+    <xacro:property name="MIN_ACCELERATION" value="-3"/> <!-- [m/s^2] -->
+    <xacro:property name="MAX_VELOCITY" value="1"/> <!-- [m/s] -->
+    <xacro:property name="MAX_ACCELERATION" value="3"/>  <!-- [m/s^2] -->
+    <xacro:property name="WHEELBASE" value="1.65"/> <!-- [m] -->
+    <xacro:property name="STEERING_LIMIT" value="0.795"/> <!-- 45 degrees in radians -->
+    <xacro:property name="TOPIC_TO_BRIDGE_ACKERMANN" value="/cmd_vel"/>
+    <xacro:property name="EFFORT_LIMIT" value="100"/>
+    <xacro:property name="VELOCITY_LIMIT" value="10"/>
     <!-- Miscellaneous materials -->
     <material name="blue"> <color rgba="0.0 0.0 0.8 1.0"/>  </material>
@@ -65,5 +74,5 @@
     <material name="black"> <color rgba="0.0 0.0 0.0 1.0"/>  </material>
     <!-- =========================================-->
-    <!-- |              ACTUAL ROBOT              |-->
+    <!-- |              ACTUAL ROBOT             |-->
     <!-- =========================================-->
     <!-- Origin of the Robot -->
@@ -100,5 +109,5 @@
         <origin xyz="${RACECAR_STEERING_HINGE_X} ${RACECAR_STEERING_HINGE_Y} ${RACECAR_STEERING_HINGE_Z}"/>
         <axis xyz="0 1 0" />
-        <limit effort="100.0" velocity="10.0" lower="-0.795" upper="+0.795"/>
+        <limit effort="${EFFORT_LIMIT}" velocity="${VELOCITY_LIMIT}" lower="-${STEERING_LIMIT}" upper="+${STEERING_LIMIT}"/>
     </joint>
     <joint name="base_chassis_to_right_steering_hinge" type="revolute">
@@ -107,5 +116,5 @@
         <origin xyz="${RACECAR_STEERING_HINGE_X} -${RACECAR_STEERING_HINGE_Y} ${RACECAR_STEERING_HINGE_Z}"/>
         <axis xyz="0 1 0" />
-        <limit effort="100.0" velocity="10.0" lower="-0.795" upper="+0.795"/>
+        <limit effort="${EFFORT_LIMIT}" velocity="${VELOCITY_LIMIT}" lower="-${STEERING_LIMIT}" upper="+${STEERING_LIMIT}"/>
     </joint>
     <joint name="base_chassis_to_left_rear_wheel" type="continuous">
@@ -114,5 +123,5 @@
         <origin xyz="${RACECAR_WHEEL_REAR_X} ${RACECAR_WHEEL_REAR_Y} ${RACECAR_WHEEL_REAR_Z}"/>
         <axis xyz="0 1 0" />
-        <limit effort="100.0" velocity="10.0"/>
+        <limit effort="${EFFORT_LIMIT}" velocity="${VELOCITY_LIMIT}"/>
     </joint>
     <joint name="base_chassis_to_right_rear_wheel" type="continuous">
@@ -121,5 +130,5 @@
         <origin xyz="${RACECAR_WHEEL_REAR_X} -${RACECAR_WHEEL_REAR_Y} ${RACECAR_WHEEL_REAR_Z}"/>
         <axis xyz="0 1 0" />
-        <limit effort="100.0" velocity="10.0"/>
+        <limit effort="${EFFORT_LIMIT}" velocity="${VELOCITY_LIMIT}"/>
     </joint>
     <!-- Left & Right Steering Hinges + Joints to wheels -->
@@ -160,5 +169,5 @@
         <origin xyz="0 0 0"/>
         <axis xyz="0 1 0" />
-        <limit effort="100.0" velocity="10.0"/>
+        <limit effort="${EFFORT_LIMIT}" velocity="${VELOCITY_LIMIT}"/>
     </joint>
     <joint name="right_steering_hinge_to_right_front_wheel" type="continuous">
@@ -167,5 +176,5 @@
         <origin xyz="0 0 0"/>
         <axis xyz="0 1 0" />
-        <limit effort="100.0" velocity="10.0"/>
+        <limit effort="${EFFORT_LIMIT}" velocity="${VELOCITY_LIMIT}"/>
     </joint>
     <!-- Front Wheels -->
@@ -247,9 +256,10 @@
         </inertial>
     </link>
+    <!-- Gazebo Ackermann Plugin-->
     <gazebo>
         <plugin
             filename="gz-sim-ackermann-steering-system"
             name="gz::sim::systems::AckermannSteering">
-            <left_joint>base_chassis_to_left_front_wheel</left_joint>
+            <left_joint>base_chassis_to_left_front_wheel</left_joint> <!-- Names defined in the joints-->
             <left_joint>base_chassis_to_left_rear_wheel</left_joint>
             <right_joint>base_chassis_to_right_front_wheel</right_joint>
@@ -257,14 +267,14 @@
             <left_steering_joint>base_chassis_to_left_steering_hinge</left_steering_joint>
             <right_steering_joint>base_chassis_to_right_steering_hinge</right_steering_joint>
-            <kingpin_width>1.0</kingpin_width>
-            <steering_limit>0.5</steering_limit>
-            <wheel_base>1.0</wheel_base>
-            <wheel_separation>1.25</wheel_separation>
-            <wheel_radius>0.3</wheel_radius>
-            <min_velocity>-1</min_velocity>
-            <max_velocity>1</max_velocity>
-            <min_acceleration>-3</min_acceleration>
-            <max_acceleration>3</max_acceleration>
-            <topic>/cmd_vel</topic>
+            <kingpin_width>${RACECAR_STEERING_HINGES_DISTANCE}</kingpin_width>
+            <steering_limit>${STEERING_LIMIT}</steering_limit>
+            <wheel_base>${WHEELBASE}</wheel_base>
+            <wheel_separation>${RACECAR_STEERING_HINGES_DISTANCE}</wheel_separation> <!-- -->
+            <wheel_radius>${WHEEL_WIDTH}</wheel_radius>
+            <min_velocity>${MIN_VELOCITY}</min_velocity>
+            <max_velocity>${MAX_VELOCITY}</max_velocity>
+            <min_acceleration>${MIN_ACCELERATION}</min_acceleration>
+            <max_acceleration>${MAX_ACCELERATION}</max_acceleration>
+            <topic>${TOPIC_TO_BRIDGE_ACKERMANN}</topic>
       </plugin>
     </gazebo>
